File: DesignTest.kicad_pcb (KiCad board)
At the start: 2 copper layers, 36.6 x 31 mm, 6 parts, among them J1 Conn_01x02, J2 Conn_01x09, J3 Conn_01x04, J4 Conn_01x02, U1 4051

Commit message: fix
Other:
- board text added: "rev fix"
- board text removed: "rev 0.1"
Changed lines of the file:
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@@
     )
   )
-  (gr_text "rev 0.1" (at 121.92 103.124) (layer F.SilkS)
+  (gr_text "rev fix" (at 121.92 103.124) (layer F.SilkS)
     (effects (font (size 1.5 1.5) (thickness 0.3)))
   )
